Commit message: changed end effector lower limit, enable jsp gui

File: ardop_description/ardop_description_01/urdf/ardop_description_01.urdf (robot description, URDF)
Before this commit: robot ardop_description_01, 11 links, 10 joints
Joints:
- joint end_effector_joint: limit lower=-1.5708 upper=1.5708 effort=30 velocity=3 -> lower=-0.6 upper=1.5708 effort=30 velocity=3
