Commit message: ROS controllers for wheels are working

File: ardop_description/ardop_description_02_experimental/urdf/ardop_description_02.urdf (robot description, URDF)
Before this commit: robot ardop_description_02, 11 links, 10 joints
Joints:
- joint lower_1_joint: origin xyz=0.0024117 0.025054 -0.070238 rpy=0 0 0 -> xyz=0.0024117 0.025054 -0.070238 rpy=0 -0.04 0
- joint upper_2_joint: origin xyz=9.3209E-05 0 -0.10405 rpy=0 0 0 -> xyz=9.3209E-05 0 -0.10405 rpy=0 0.04 0
