Commit message: Initial commit

File: ardop_description/urdf/ardop_description.urdf (robot description, URDF)
Before this commit: robot ardop, 13 links, 12 joints
Links:
- removed link base_link
- removed link lower_3_link
- removed link odom
- removed link upper_2_link
- added link chassis_link, mass 13.474; collision mesh filename=package://ardop_description/meshes/chassis_link.STL; visual mesh filename=package://ardop_description/meshes/chassis_link.STL
- added link ee_pitch_link, mass 0.039125; collision mesh filename=package://ardop_description/meshes/ee_pitch_link.STL; visual mesh filename=package://ardop_description/meshes/ee_pitch_link.STL
- added link ee_roll_link, mass 0.15479; collision mesh filename=package://ardop_description/meshes/ee_roll_link.STL; visual mesh filename=package://ardop_description/meshes/ee_roll_link.STL
- link end_effector_link: mass 0.010303 -> 0.050107
- link lower_1_link: mass 0.2241 -> 0.51863
- link lower_2_link: mass 0.078 -> 0.50115
- link shoulder_1_link: mass 0.239718 -> 0.38511
- link upper_1_link: mass 0.158253 -> 0.65289
- link wheel_back_left_link: mass 0.4 -> 0.32836
- link wheel_back_right_link: mass 0.4 -> 0.32836
- link wheel_front_left_link: mass 0.4 -> 0.32836
- link wheel_front_right_link: mass 0.4 -> 0.32836
Joints:
- removed joint lower_3_joint
- removed joint odom_joint
- removed joint upper_2_joint
- added joint ee_pitch_joint: type revolute, parent lower_2_link, child ee_pitch_link, origin xyz=0.011877 -0.028151 0.11857 rpy=-1.5708 0 -3.1416, axis 0 0 1, limit effort=0 velocity=0
- added joint ee_roll_joint: type revolute, parent ee_pitch_link, child ee_roll_link, origin xyz=-0.0311 -0.014379 0.017 rpy=-1.5708 0 1.5708, axis 0 0 1, limit effort=0 velocity=0
- joint end_effector_joint: axis 1 0 0 -> 0 0 1; limit lower=-0.6 upper=1.5708 effort=300 velocity=3 -> effort=0 velocity=0; origin xyz=0.020065 0.0095794 -0.03 rpy=0 0 0 -> xyz=0.02055 0.030611 0.034 rpy=-1.5708 0 -1.5708; parent lower_3_link -> ee_roll_link
- joint lower_1_joint: axis 0 1 0 -> 0 0 1; limit lower=-1.5708 upper=1.5708 effort=300 velocity=3 -> effort=0 velocity=0; origin xyz=0.0024117 0.025054 -0.070238 rpy=0 0 0 -> xyz=0.00017493 -0.17353 -0.025178 rpy=3.1416 0 -1.5708; parent upper_2_link -> upper_1_link
- joint lower_2_joint: axis 0 0 1 -> 0 0 -1; limit lower=-1.5708 upper=1.5708 effort=300 velocity=3 -> effort=0 velocity=0; origin xyz=0 -0.030211 -0.12948 rpy=0 0 0 -> xyz=0.12948 0 -0.030211 rpy=-1.5708 0 -1.5708
- joint shoulder_1_joint: axis 1 0 0 -> 0 0 1; limit lower=-1.5708 upper=1.5708 effort=300 velocity=3 -> effort=0 velocity=0; origin xyz=-0.0281 -0.25288 0.504 rpy=0 0 0 -> xyz=-0.002 -0.25288 0.5401 rpy=0 0 0; parent base_link -> chassis_link
- joint upper_1_joint: axis 0 1 0 -> 0 0 -1; limit lower=-1.5708 upper=1.5708 effort=300 velocity=3 -> effort=0 velocity=0; origin xyz=0.027024 -0.075963 0.0044026 rpy=0 -0.034323 0 -> xyz=0.0027 -0.075963 -0.026697 rpy=1.5708 0 0
- joint wheel_back_left_joint: limit effort=100 velocity=100 -> (none); origin xyz=-0.2 0.1895 0.05 rpy=0 0 0 -> xyz=-0.2 0.1995 0.05 rpy=0 0 0; parent base_link -> chassis_link
- joint wheel_back_right_joint: limit effort=100 velocity=100 -> (none); origin xyz=-0.2 -0.1895 0.05 rpy=0 0 0 -> xyz=-0.2 -0.1995 0.05 rpy=0 0 0; parent base_link -> chassis_link
- joint wheel_front_left_joint: limit effort=100 velocity=100 -> (none); origin xyz=0.03 0.1895 0.05 rpy=0 0 0 -> xyz=0.03 0.1995 0.05 rpy=0 0 0; parent base_link -> chassis_link
- joint wheel_front_right_joint: limit effort=100 velocity=100 -> (none); origin xyz=0.03 -0.1895 0.05 rpy=0 0 0 -> xyz=0.03 -0.1995 0.05 rpy=0 0 0; parent base_link -> chassis_link

Commit message: IK using KDL is working

File: ardop_description/urdf/ardop_description.urdf (robot description, URDF)
Before this commit: robot ardop_description, 12 links, 11 joints
Links:
- added link odom
- link chassis_link: mass 13.474 -> 6
- link ee_pitch_link: mass 0.039125 -> 0.07
- link ee_roll_link: mass 0.15479 -> 0.11
- link end_effector_link: mass 0.050107 -> 0.010303
- link lower_1_link: mass 0.51863 -> 0.2241
- link lower_2_link: mass 0.50115 -> 0.143
- link shoulder_1_link: mass 0.38511 -> 0.239718
- link upper_1_link: mass 0.65289 -> 0.169459
- link wheel_back_left_link: mass 0.32836 -> 0.4
- link wheel_back_right_link: mass 0.32836 -> 0.4
- link wheel_front_left_link: mass 0.32836 -> 0.4
- link wheel_front_right_link: mass 0.32836 -> 0.4
Joints:
- added joint odom_joint: type fixed, parent odom, child chassis_link
- joint ee_pitch_joint: limit effort=0 velocity=0 -> lower=-0.785398 upper=2.35619 effort=300 velocity=3
- joint ee_roll_joint: limit effort=0 velocity=0 -> lower=-1.5708 upper=1.5708 effort=300 velocity=3
- joint end_effector_joint: limit effort=0 velocity=0 -> lower=-0.6 upper=1.5708 effort=300 velocity=3
- joint lower_1_joint: limit effort=0 velocity=0 -> lower=-1.5708 upper=1.5708 effort=300 velocity=3
- joint lower_2_joint: limit effort=0 velocity=0 -> lower=-1.5708 upper=1.5708 effort=300 velocity=3
- joint shoulder_1_joint: limit effort=0 velocity=0 -> lower=-1.5708 upper=1.5708 effort=300 velocity=3
- joint upper_1_joint: limit effort=0 velocity=0 -> lower=-1.5708 upper=1.5708 effort=300 velocity=3
- joint wheel_back_left_joint: limit (none) -> effort=100 velocity=100; origin xyz=-0.2 0.1995 0.05 rpy=0 0 0 -> xyz=-0.2 0.1895 0.05 rpy=0 0 0
- joint wheel_back_right_joint: limit (none) -> effort=100 velocity=100; origin xyz=-0.2 -0.1995 0.05 rpy=0 0 0 -> xyz=-0.2 -0.1895 0.05 rpy=0 0 0
- joint wheel_front_left_joint: limit (none) -> effort=100 velocity=100; origin xyz=0.03 0.1995 0.05 rpy=0 0 0 -> xyz=0.03 0.1895 0.05 rpy=0 0 0
- joint wheel_front_right_joint: limit (none) -> effort=100 velocity=100; origin xyz=0.03 -0.1995 0.05 rpy=0 0 0 -> xyz=0.03 -0.1895 0.05 rpy=0 0 0

Commit message: Fixed inertia for Gazebo

File: ardop_description/urdf/ardop_description.urdf (robot description, URDF)
Before this commit: robot ardop, 13 links, 12 joints
Links:
- link ee_pitch_link: mass 0.07 -> 0.1
- link ee_roll_link: mass 0.11 -> 0.1
- link end_effector_link: mass 0.010303 -> 0.1
- link lower_1_link: mass 0.2241 -> 0.1
- link lower_2_link: mass 0.143 -> 0.1
- link shoulder_1_link: mass 0.239718 -> 0.1
- link upper_1_link: mass 0.169459 -> 0.1
